File: chandra_queenofnight.kicad_pcb (KiCad board)
At the start: 2 copper layers, 88 parts, among them IC1 bp060674p12, IC2 bp060674p12, J1 B5B-XH-A, J2 Screw_Terminal_01x03, J3 B5B-XH-A, J4 B2B-XH-A__LF__SN_, J5 B2B-XH-A__LF__SN_, J6 B4B-XH-A_LF__SN_, J7 51494-2, J8 51494-2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

Commit message: Initialtes
Parts:
- removed R_dac2_pup_scl1, R_dac2_pup_sda1: 4.7k, Resistor_THT:R_Axial_DIN0207_L6.3mm_D2.5mm_P7.62mm_Horizontal
- added D5: D_Zener, Diode_THT:D_5KP_P12.70mm_Horizontal, F.Cu at (250.1, 99.5)
- added T1: 7508112339, kaam25_footprints_symbol:WE-OLTI_EE20_10_6_L22.2W26H16.5, F.Cu at (241.2, 52.6)
- added U5: UC3842N, kaam25_footprints_symbol:DIP794W45P254L959H508Q8, F.Cu at (222.1, 148.5)
- moved C3 132.0 mm to (264.6, 43.4), turned to 180 degrees
- moved R_dac1_pup_scl1 111.7 mm to (44.7, 180.2), turned to -90 degrees
- moved R_dac1_pup_sda1 109.8 mm to (52.1, 188.0), turned to 90 degrees
- moved C_T1 109.5 mm to (229.4, 146.3), turned to -90 degrees
- moved Q1 109.3 mm to (249.8, 140.0), turned to 180 degrees
- moved C_vcc1 108.0 mm to (225.0, 134.3), turned to -90 degrees
- moved R_sense1 106.5 mm to (234.3, 152.4)
- moved U1 103.7 mm to (150.1, 166.8)
- moved J1 103.7 mm to (133.0, 168.7)
- moved J3 103.7 mm to (133.0, 175.9)
- moved J6 103.7 mm to (131.7, 183.2)
- moved D1 103.7 mm to (143.6, 174.1)
- moved D2 103.7 mm to (149.6, 174.1)
- moved U3 103.7 mm to (150.1, 170.5)
- moved J4 103.7 mm to (170.6, 168.7)
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Connections:
- R_dac1_pup_scl1 pad 1: 3.3V -> Net-(U2-IO21)
- R_dac1_pup_scl1 pad 2: Net-(U2-IO21) -> 3.3V
Routing:
- net GND: track 0.00 -> 42.2 mm
- net VCC: track 0.00 -> 24.2 mm
- net Net-(C_filter2-Pad1): track 0.00 -> 18.4 mm
- net Net-(D_snub1-A): track 0.00 -> 17.7 mm
- net Net-(D_snub1-K): track 0.00 -> 15.8 mm
- net Net-(D_fastSwitchig_out2-A): track 0.00 -> 11.4 mm
- net 12V: track 0.00 -> 10.3 mm
- net Net-(D_fastSwitchig_out2-K): track 0.00 -> 7.18 mm
- net Net-(D_fastSwitchig_out1-A): track 0.00 -> 6.51 mm
- net GND1: track 0.00 -> 6.14 mm

Commit message: Initialtes 130426
Parts:
- removed D5: D_Zener, Diode_THT:D_5KP_P12.70mm_Horizontal
- removed FL1: Choke_CommonMode_PulseElectronics_PH9455x826NL, Inductor_THT:L_CommonMode_PulseElectronics_PH9455xxx6NL_2
- removed R_oled_pup_scl1, R_oled_pup_sda1: 4.7k, Resistor_THT:R_Axial_DIN0207_L6.3mm_D2.5mm_P7.62mm_Horizontal
- removed U8: DM-OLED096-636, kaam25_footprints_symbol:MODULE_DM-OLED096-636
- R_startUp1, R_startUp2: value 68k -> 83k
- R_startUp3: value 68k -> 1.26k
- moved U11 124.3 mm to (270.5, 75.7), turned to -90 degrees
- moved C_bypass1 114.5 mm to (132.8, 153.6)
- moved R_up1 104.3 mm to (262.6, 58.2), turned to -90 degrees
- moved C_bs1 103.1 mm to (137.3, 139.1), turned to 90 degrees
- moved J5 97.1 mm to (73.8, 183.7), turned to -90 degrees
- moved R_led1 95.6 mm to (267.2, 58.8)
- moved R11 93.1 mm to (61.7, 190.8), turned to 180 degrees
- moved RV1 89.4 mm to (220.6, 128.4), turned to 180 degrees
- moved C_filter2 85.1 mm to (193.6, 114.7)
- moved C_filter1 84.4 mm to (157.0, 133.4), turned to -90 degrees
- moved C_op_5 83.1 mm to (139.4, 129.0)
- moved C_decoup_12V2 81.2 mm to (39.8, 105.5), turned to -90 degrees
- moved C_comp1 80.0 mm to (163.4, 133.5), turned to -90 degrees
- moved U10 78.0 mm to (271.3, 62.4), turned to -90 degrees
- moved R_down1 73.6 mm to (257.8, 70.8), turned to 90 degrees
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Connections:
- D3 pad 2: Net-(D3-Pad2) -> /sunny_sheet_1/N
- D3 pad 4: Net-(D3-Pad4) -> /sunny_sheet_1/L
- R_startUp2 pad 1: Net-(R_startUp2-Pad1) -> VCC
- R_startUp3 pad 1: VCC -> GND1
- R_startUp3 pad 2: Net-(R_startUp2-Pad1) -> VCC
Routing:
- net Net-(IC1-HV): track 0.00 -> 37.6 mm
- net Net-(IC1-GND_2): track 0.00 -> 36.5 mm
- net Net-(IC2-GND_2): track 0.00 -> 33.1 mm
- net Net-(IC2-HV): track 0.00 -> 32.5 mm

Commit message: Initialtes
Parts:
- added U8: DM-OLED096-636, kaam25_footprints_symbol:MODULE_DM-OLED096-636, F.Cu at (267.0, 32.4)
- U2: footprint kaam25_footprints_symbol:MODULE_DEVKIT_V1_ESP32-WROOM-32 -> kaam25:MODULE_DEVKIT_V1_ESP32-WROOM-32
- moved J5 225.7 mm to (273.1, 77.9)
- moved R11 225.7 mm to (261.0, 85.0)
- moved R_dac1_pup_scl1 225.7 mm to (244.0, 74.4)
- moved R_dac1_pup_sda1 225.7 mm to (251.4, 82.2)
- moved U7 225.7 mm to (260.0, 78.2)
- moved U6 225.7 mm to (261.3, 69.5)
- moved U2 195.1 mm to (228.5, 144.0), turned to 90 degrees
- moved C3 181.0 mm to (83.6, 41.9)
- moved C_bp_1 181.0 mm to (50.6, 81.6)
- moved C_snub1 181.0 mm to (42.6, 48.6)
- moved D4 181.0 mm to (37.0, 83.9)
- moved D_fastSwitchig_out2 181.0 mm to (60.4, 66.5)
- moved D_snub1 181.0 mm to (42.8, 44.3)
- moved R_led1 181.0 mm to (86.2, 57.4)
- moved R_snub1 181.0 mm to (37.1, 67.1)
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Connections:
- J1 pad 1: Net-(U2-IO27) -> Net-(U2-IO26)
- J1 pad 2: Net-(U2-IO32) -> Net-(U2-IO35)
- J1 pad 3: Net-(U2-IO34) -> Net-(U2-SENSOR_VN)
- J3 pad 3: Net-(U2-IO26) -> Net-(U2-IO25)
- J3 pad 4: Net-(U2-IO19) -> Net-(U2-GND2)
- J3 pad 5: Net-(U2-IO13) -> Net-(U2-GND1)
- J4 pad 2: Net-(U2-IO4) -> Net-(U2-IO16)
- J5 pad 1: Net-(U2-IO23) -> Net-(U2-GND3)
- J6 pad 2: Net-(U2-IO21) -> Net-(U2-RXD0)
- J6 pad 3: Net-(U2-IO22) -> Net-(U2-IO23)
- R1 pad 2: Net-(U2-IO35) -> Net-(U2-IO34)
- R2 pad 2: Net-(U2-SENSOR_VP) -> Net-(U2-EN)
- R3 pad 1: Net-(U2-IO35) -> Net-(U2-IO34)
- R4 pad 1: Net-(U2-SENSOR_VP) -> Net-(U2-EN)
- R5 pad 2: Net-(U2-IO33) -> Net-(U2-IO32)
- R6 pad 2: Net-(U2-SENSOR_VN) -> Net-(U2-SENSOR_VP)
- R7 pad 1: Net-(U2-IO33) -> Net-(U2-IO32)
- R8 pad 1: Net-(U2-SENSOR_VN) -> Net-(U2-SENSOR_VP)
- R_dac1_pup_scl1 pad 1: Net-(U2-IO21) -> Net-(U2-RXD0)
- R_dac1_pup_sda1 pad 2: Net-(U2-IO22) -> Net-(U2-IO23)
- U2 pad 1: 3.3V -> unconnected-(U2-3V3-Pad1)
- U2 pad 11: Net-(U2-IO27) -> unconnected-(U2-IO27-Pad11)
- U2 pad 13: unconnected-(U2-IO12-Pad13) -> GND2
- U2 pad 14: GND2 -> Net-(U2-GND1)
- U2 pad 15: Net-(U2-IO13) -> unconnected-(U2-IO13-Pad15)
- U2 pad 2: unconnected-(U2-EN-Pad2) -> Net-(U2-EN)
- U2 pad 26: Net-(U2-IO4) -> unconnected-(U2-IO4-Pad26)
- U2 pad 27: unconnected-(U2-IO16-Pad27) -> Net-(U2-IO16)
- U2 pad 31: Net-(U2-IO19) -> unconnected-(U2-IO19-Pad31)
- U2 pad 32: unconnected-(U2-GND2-Pad32) -> Net-(U2-GND2)
- U2 pad 33: Net-(U2-IO21) -> unconnected-(U2-IO21-Pad33)
- U2 pad 34: unconnected-(U2-RXD0-Pad34) -> Net-(U2-RXD0)
- U2 pad 36: Net-(U2-IO22) -> unconnected-(U2-IO22-Pad36)
- U2 pad 38: unconnected-(U2-GND3-Pad38) -> Net-(U2-GND3)
- U2 pad 8: Net-(U2-IO33) -> unconnected-(U2-IO33-Pad8)
- U2 pad 9: unconnected-(U2-IO25-Pad9) -> Net-(U2-IO25)
- U6 pad 4: Net-(U2-IO22) -> Net-(U2-IO23)
- U6 pad 5: Net-(U2-IO21) -> Net-(U2-RXD0)
- U7 pad 4: Net-(U2-IO22) -> Net-(U2-IO23)
- U7 pad 5: Net-(U2-IO21) -> Net-(U2-RXD0)
Routing:
- net GND1: track 6.14 -> 55.6 mm
- net GND: track 42.2 -> 86.3 mm
- net 12V: track 10.3 -> 51.8 mm
- net VCC: track 24.2 -> 55.3 mm
- net Net-(D6-K): track 0.00 -> 28.3 mm
- net Net-(U11-K): track 0.00 -> 12.3 mm
- net Net-(U4-BS): track 0.00 -> 10.7 mm
- net Net-(R_led1-Pad2): track 0.00 -> 10.1 mm
- net 5V: track 0.00 -> 8.82 mm
- net V_fb: track 0.00 -> 8.07 mm
- net Net-(U11-REF): track 0.00 -> 7.01 mm
- net Net-(R_startUp1-Pad1): track 0.00 -> 3.49 mm
- net 3.3V: track 0.00 -> 2.93 mm
- added copper zone on F.Cu, net Net-(D6-K)
Other:
- copper layers 2 -> 4

Commit message: Initialtes gndplane
Parts:
- added C_decoup_3V2: 10u, Capacitor_THT:CP_Radial_D5.0mm_P2.00mm, F.Cu at (158.2, 167.1)
- J2: footprint TerminalBlock_MetzConnect:TerminalBlock_MetzConnect_360291_1x01_Horizontal_ScrewM3.0_Boxed -> TerminalBlock_MetzConnect:TerminalBlock_MetzConnect_Type011_RT05503HBLC_1x03_P5.00mm_Horizontal
- moved D1 159.3 mm to (241.6, 45.8)
- moved D2 159.3 mm to (247.6, 45.8)
- moved RV1 146.7 mm to (40.4, 17.0), turned to 0 degrees
- moved J5 136.8 mm to (144.5, 124.6), turned to 180 degrees
- moved C_X1 132.8 mm to (40.1, 23.1), turned to -90 degrees
- moved C_Y_2 123.3 mm to (52.0, 24.4), turned to 180 degrees
- moved C_filter2 115.1 mm to (65.2, 26.5), turned to -90 degrees
- moved R11 114.3 mm to (153.7, 124.4)
- moved U6 110.0 mm to (162.6, 118.0)
- moved J2 108.1 mm to (20.6, 24.7), turned to -90 degrees
- moved TH1 102.3 mm to (56.5, 33.0), turned to 90 degrees
- moved D3 100.2 mm to (52.4, 37.6), turned to 180 degrees
- moved X1 92.5 mm to (114.4, 127.0), turned to 0 degrees
- moved R_dac1_pup_scl1 91.8 mm to (166.8, 124.0), turned to 180 degrees
- moved U7 89.3 mm to (179.9, 117.8), turned to 90 degrees
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Connections:
- J1 pad 3: Net-(U2-SENSOR_VN) -> Net-(U2-IO33)
- J3 pad 3: Net-(U2-IO25) -> Net-(U2-GND2)
- J3 pad 4: Net-(U2-GND2) -> Net-(U2-IO12)
- J3 pad 5: Net-(U2-GND1) -> Net-(U2-IO25)
- R2 pad 2: Net-(U2-EN) -> Net-(U2-SENSOR_VN)
- R4 pad 1: Net-(U2-EN) -> Net-(U2-SENSOR_VN)
- U2 pad 1: unconnected-(U2-3V3-Pad1) -> Net-(U2-3V3)
- U2 pad 13: GND2 -> Net-(U2-IO12)
- U2 pad 14: Net-(U2-GND1) -> GND2
- U2 pad 2: Net-(U2-EN) -> Net-(U2-3V3)
- U2 pad 8: unconnected-(U2-IO33-Pad8) -> Net-(U2-IO33)
Routing:
- net Net-(IC1-HV): track 37.6 -> 39.2 mm
- added copper zone on F.Cu, net GND
- removed copper zone on F.Cu, net Net-(D6-K)

Commit message: Initialtes apr21
Parts:
- R_comp1: value 1.5k -> 10k
- moved U8 220.3 mm to (103.0, 179.6)
- moved R12 171.2 mm to (180.1, 62.6)
- moved D1 164.8 mm to (130.7, 167.6)
- moved D2 164.8 mm to (136.7, 167.6)
- moved U3 160.1 mm to (150.9, 167.6)
- moved U1 152.5 mm to (166.6, 167.5)
- moved J4 148.9 mm to (89.5, 46.4)
- moved R2 145.7 mm to (169.3, 29.4)
- moved R3 145.7 mm to (151.2, 18.8)
- moved R7 145.7 mm to (165.7, 18.6)
- moved R8 145.7 mm to (164.4, 36.8)
- moved C_decoup_3V2 145.7 mm to (141.4, 22.4)
- moved R1 145.7 mm to (155.3, 26.4)
- moved R4 145.7 mm to (174.1, 36.9)
- moved R5 145.7 mm to (160.5, 26.4)
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Connections:
- C_T1 pad 1: GND1 -> GND
- C_bypass1 pad 1: GND1 -> GND
- C_comp2 pad 1: GND1 -> GND
- C_filter3 pad 2: GND1 -> GND
- R_Fb1 pad 1: GND1 -> GND
- R_sense1 pad 2: GND1 -> GND
- R_startUp3 pad 1: GND1 -> GND
- U10 pad 3: GND1 -> GND
- U5 pad 5: GND1 -> GND
Routing:
- net GND: track 86.3 -> 27.1 mm
- net GND1: track 55.6 -> 0.00 mm
- net VCC: track 55.3 -> 0.00 mm
- net 12V: track 51.8 -> 6.41 mm
- net Net-(IC1-HV): track 39.2 -> 0.00 mm
- net Net-(IC1-GND_2): track 36.5 -> 0.00 mm
- net Net-(IC2-GND_2): track 33.1 -> 0.00 mm
- net Net-(IC2-HV): track 32.5 -> 0.00 mm
- net Net-(C_filter2-Pad1): track 18.4 -> 0.17 mm
- net Net-(D_snub1-A): track 17.7 -> 0.00 mm
- net Net-(D_snub1-K): track 15.8 -> 0.00 mm
- net Net-(U11-K): track 12.3 -> 0.00 mm
- net Net-(D_fastSwitchig_out2-A): track 11.4 -> 0.00 mm
- net Net-(R_led1-Pad2): track 10.1 -> 0.00 mm
- net Net-(D_fastSwitchig_out2-K): track 7.18 -> 0.00 mm
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- removed copper zone on F.Cu, net GND
Other:
- copper layers 4 -> 2

Commit message: Initialtes apr22
Parts:
- added J10: B2B-XH-A, kaam25:B2P-VH, F.Cu at (275.5, 192.2)
- added J9: B2B-XH-A, kaam25:B2P-VH, F.Cu at (133.0, 59.0)
- J1, J3: value B5B-XH-A -> B5B-XH-A_rotataryKnob
- J4, J5: value B2B-XH-A__LF__SN_ -> B2B-XH-A__LF__SN_ledTwoTerminal
- J6: value B4B-XH-A_LF__SN_ -> B4B-XH-A_LF__SN_oled_display; moved to B.Cu
- moved R12 99.9 mm to (81.3, 47.5), turned to 90 degrees
- moved J6 94.7 mm to (90.7, 61.0), turned to 90 degrees
- moved R1 86.4 mm to (160.7, 112.7)
- moved R3 81.7 mm to (164.2, 99.5), turned to 0 degrees
- moved R7 75.8 mm to (164.4, 94.4), turned to 0 degrees
- moved J1 60.2 mm to (166.6, 128.8), turned to 90 degrees
- moved X1 59.3 mm to (122.1, 71.8), turned to -90 degrees
- moved R5 56.5 mm to (160.8, 82.9), turned to -90 degrees
- moved J3 56.2 mm to (182.7, 129.2), turned to -90 degrees
- moved U6 54.8 mm to (156.1, 102.1)
- moved C_decoup_3V1 51.5 mm to (80.2, 23.9)
- moved R_dac1_pup_scl1 48.8 mm to (150.9, 105.8), turned to 90 degrees
- moved R11 42.6 mm to (147.2, 133.7), turned to 90 degrees
- moved C_decoup_12V1 38.7 mm to (171.2, 84.1)
- moved J5 34.7 mm to (154.1, 133.3)
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
Commit message: Initialtes apr24
Parts:
- added X3: B2P-VH, Connector_JST:JST_VH_B2P-VH-B_1x02_P3.96mm_Vertical, F.Cu at (106.8, 85.0)
- J6: moved to F.Cu
- moved J3 133.3 mm to (78.1, 46.5)
- moved J10 128.4 mm to (154.0, 150.6)
- moved C_bypass1 123.5 mm to (23.6, 74.3)
- moved J1 97.3 mm to (117.4, 44.9)
- moved R_Fb1 97.0 mm to (23.1, 103.8)
- moved U6 87.2 mm to (77.8, 63.5), turned to 90 degrees
- moved R_dac1_pup_scl1 82.0 mm to (141.2, 24.4), turned to -90 degrees
- moved U7 76.6 mm to (77.8, 57.8)
- moved J6 55.4 mm to (135.1, 28.1), turned to -90 degrees
- moved R_up1 48.7 mm to (83.4, 69.5)
- moved R_down1 47.7 mm to (78.0, 78.7)
- moved C_in1 46.0 mm to (129.7, 97.3)
- moved U9 46.0 mm to (123.6, 98.5)
- moved C_out1 46.0 mm to (119.8, 93.2)
- moved C_decoup_3V1 44.0 mm to (124.2, 27.1)
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Connections:
- net Net-(IC1-VSET) renamed /chandu_sheet_2/vset_a
- net Net-(IC1-~{ON}) renamed /chandu_sheet_2/\ON_a
- net Net-(IC2-VSET) renamed /chandu_sheet_2/vset_b
- net Net-(IC2-~{ON}) renamed /chandu_sheet_2/\ON_b
- net Net-(U2-GND2) renamed /chandu_sheet_2/SW_B
- net Net-(U2-IO16) renamed /chandu_sheet_2/led_b
- net Net-(U2-IO23) renamed /chandu_sheet_2/sda_a
- net Net-(U2-IO26) renamed /chandu_sheet_2/CLK_a
- net Net-(U2-IO32) renamed /chandu_sheet_2/adc_I_a
- net Net-(U2-IO33) renamed /chandu_sheet_2/SW_a
- net Net-(U2-IO34) renamed /chandu_sheet_2/adc_V_a
- net Net-(U2-IO35) renamed /chandu_sheet_2/DT_a
- net Net-(U2-RXD0) renamed /chandu_sheet_2/scl_a
- net Net-(U2-SENSOR_VN) renamed /chandu_sheet_2/adc_I_b
- net Net-(U2-SENSOR_VP) renamed /chandu_sheet_2/adc_V_b
- C_comp1 pad 2: GND -> GND1
- C_decoup_12V1 pad 1: GND -> GND1
- C_decoup_12V2 pad 1: GND -> GND1
- C_decoup_3V1 pad 2: GND2 -> GND1
- C_decoup_3V2 pad 1: GND2 -> GND1
- C_filter1 pad 2: GND -> GND1
- C_op_5 pad 1: GND -> GND1
- D6 pad 2: GND -> GND1
- IC1 pad 1: GND -> GND1
- IC1 pad 7: Net-(IC1-REF) -> /chandu_sheet_2/ref_b
- IC1 pad 8: GND -> GND1
- IC2 pad 1: GND -> GND1
- IC2 pad 7: Net-(IC2-REF) -> /chandu_sheet_2/ref_b
- IC2 pad 8: GND -> GND1
- J1 pad 4: 3.3V -> Net-(U2-3V3)
- J1 pad 5: GND2 -> GND1
- J3 pad 1: GND -> GND1
- J3 pad 4: Net-(U2-IO12) -> /chandu_sheet_2/DT_b
- J3 pad 5: Net-(U2-IO25) -> /chandu_sheet_2/CLK_b
- J5 pad 1: Net-(U2-GND3) -> /chandu_sheet_2/led_a
- J6 pad 4: GND -> GND1
- R1 pad 1: GND -> GND1
- R2 pad 1: GND -> GND1
- R5 pad 1: GND -> GND1
- R6 pad 1: GND -> GND1
- R9 pad 1: GND -> GND1
- U2 pad 13: Net-(U2-IO12) -> unconnected-(U2-IO12-Pad13)
- U2 pad 14: GND2 -> GND1
- U2 pad 30: unconnected-(U2-IO18-Pad30) -> /chandu_sheet_2/CLK_b
- U2 pad 31: unconnected-(U2-IO19-Pad31) -> /chandu_sheet_2/DT_b
- U2 pad 33: unconnected-(U2-IO21-Pad33) -> /chandu_sheet_2/led_a
- U2 pad 38: Net-(U2-GND3) -> unconnected-(U2-GND3-Pad38)
- U2 pad 9: Net-(U2-IO25) -> unconnected-(U2-IO25-Pad9)
- U4 pad 2: GND -> GND1
- U4 pad 6: GND -> GND1
- U4 pad 7: GND -> GND1
- U6 pad 2: GND -> GND1
- U6 pad 3: Net-(IC1-REF) -> /chandu_sheet_2/ref_b
- U6 pad 6: GND -> GND1
- U7 pad 2: GND -> GND1
- U7 pad 3: Net-(IC2-REF) -> /chandu_sheet_2/ref_b
Routing:
- net Net-(D6-K): track 28.3 -> 0.00 mm
- net GND: track 27.1 -> 0.00 mm
- net v_opto: track 0.00 -> 22.3 mm
- net Net-(Q1-G): track 0.00 -> 21.9 mm
- net Net-(C_filter2-Pad1): track 0.17 -> 21.8 mm
- net Net-(Q1-S): track 0.00 -> 19.8 mm
- net Net-(U5-VREF): track 0.00 -> 17.6 mm
- net GND1: track 0.00 -> 15.3 mm
- net Net-(D_snub1-K): track 0.00 -> 15.0 mm
- net Net-(D_snub1-A): track 0.00 -> 12.4 mm
- net Net-(D_fastSwitchig_out2-A): track 0.00 -> 12.1 mm
- net Net-(U5-RT/CT): track 0.04 -> 11.9 mm
- net Net-(U4-BS): track 10.7 -> 0.00 mm
- net Net-(C_comp2-Pad2): track 0.00 -> 9.81 mm
- net Net-(D_fastSwitchig_out1-A): track 0.00 -> 8.78 mm
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- added copper zone on B.Cu, net GND
- added copper zone on F.Cu, net GND

Commit message: Initialtes apr26
Parts:
- moved J5 125.6 mm to (78.5, 33.0), turned to -90 degrees
- moved R_dac1_pup_scl1 90.3 mm to (57.8, 59.0), turned to 90 degrees
- moved J6 75.2 mm to (65.1, 55.4), turned to 90 degrees
- moved R_dac1_pup_sda1 71.6 mm to (62.9, 43.4), turned to 180 degrees
- moved R12 65.2 mm to (71.7, 21.9)
- moved J4 63.8 mm to (78.2, 23.8), turned to 90 degrees
- moved J10 62.3 mm to (130.6, 92.8)
- moved R11 35.2 mm to (128.3, 104.0)
- moved R_Fb1 30.2 mm to (43.7, 81.7), turned to -90 degrees
- moved C_in1 18.2 mm to (128.8, 79.2)
- moved R5 16.7 mm to (136.9, 77.4)
- moved C_out1 14.9 mm to (118.2, 78.4)
- moved TH1 14.9 mm to (38.9, 40.8)
- moved U9 12.5 mm to (122.7, 86.0)
- moved C_Y_2 12.0 mm to (23.9, 45.8)
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Connections:
- net Net-(IC1-IMON) renamed /chandu_sheet_2/i_mon_a
- net Net-(IC1-VMON) renamed /chandu_sheet_2/v_mon_a
- net Net-(IC2-IMON) renamed /chandu_sheet_2/i_mon_b
- net Net-(IC2-VMON) renamed /chandu_sheet_2/v_mon_b
- IC1 pad 7: /chandu_sheet_2/ref_b -> /chandu_sheet_2/ref_a
- U6 pad 3: /chandu_sheet_2/ref_b -> /chandu_sheet_2/ref_a
Routing:
- net /sunny_sheet_1/N: track 0.00 -> 58.5 mm
- net /sunny_sheet_1/G: track 0.00 -> 36.0 mm
- net 12V: track 0.00 -> 30.6 mm
- net /sunny_sheet_1/L: track 0.00 -> 29.8 mm
- net Net-(C_filter2-Pad1): track 21.8 -> 49.8 mm
- net 3.3V: track 0.00 -> 25.7 mm
- net VCC: track 0.00 -> 23.7 mm
- net GND1: track 15.3 -> 0.45 mm
- net Net-(U2-3V3): track 0.00 -> 13.7 mm
- net Net-(R_led1-Pad2): track 0.00 -> 13.3 mm
- net Net-(Q1-S): track 19.8 -> 31.9 mm
- net /chandu_sheet_2/led_b: track 0.00 -> 11.6 mm
- net Net-(U5-OUT): track 0.00 -> 11.4 mm
- net /chandu_sheet_2/DT_a: track 0.00 -> 11.3 mm
- net /chandu_sheet_2/sda_a: track 0.00 -> 11.1 mm
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- removed copper zone on B.Cu, net GND
- removed copper zone on F.Cu, net GND
