File: chandra_queenofnight.kicad_pcb (KiCad board)
At the start: 2 copper layers, 89 parts, among them IC1 bp060674p12, IC2 bp060674p12, J1 B5B-XH-A_rotataryKnob, J10 B2B-XH-A, J2 Screw_Terminal_01x03, J3 B5B-XH-A_rotataryKnob, J4 B2B-XH-A__LF__SN_ledTwoTermin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, J5 B2B-XH-A__LF__SN_ledTwoTermin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, J6 B4B-XH-A_LF__SN_oled_display, J7 51494-2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

Commit message: Initialtes draft1
Parts:
- removed C_decoup_3V1: 10u, Capacitor_THT:CP_Radial_D5.0mm_P2.00mm
- removed J10: B2B-XH-A, kaam25:B2P-VH
- added X4: B2P-VH, Connector_JST:JST_VH_B2P-VH-B_1x02_P3.96mm_Vertical, F.Cu at (128.4, 36.2)
- added X5: B2P-VH, Connector_JST:JST_VH_B2P-VH-B_1x02_P3.96mm_Vertical, F.Cu at (153.5, 122.8)
- moved R11 36.3 mm to (126.6, 67.8)
- moved J8 26.1 mm to (217.2, 49.1)
- moved J7 25.4 mm to (218.2, 94.3)
- moved R_dac1_pup_scl1 16.0 mm to (51.1, 44.5), turned to 0 degrees
- moved R_dac1_pup_sda1 12.8 mm to (51.3, 49.0), turned to -90 degrees
- moved J5 9.35 mm to (69.1, 33.1)
- moved R_down1 7.29 mm to (71.2, 76.1)
- moved R_up1 6.77 mm to (76.8, 71.2)
- moved C_decoup_12V1 3.84 mm to (143.0, 93.2)
- moved R5 3.06 mm to (136.7, 80.5)
- moved C_filter2 2.58 mm to (53.9, 37.8)
- moved C_in1 2.31 mm to (129.1, 81.5)
- moved C_comp2 2.05 mm to (27.3, 97.0)
- moved U9 1.57 mm to (121.2, 86.0)
- moved U6 0.75 mm to (77.8, 64.3)
- renumbered C_decoup_3V2 to C_decoup_3V3_2
Connections:
- net VCC renamed /sunny_sheet_1/v_startup
- C_decoup_3V3_2 pad 2: Net-(U2-3V3) -> /chandu_sheet_2/3v3_esp32
- J1 pad 4: Net-(U2-3V3) -> /chandu_sheet_2/3v3_esp32
- J3 pad 2: 3.3V -> /chandu_sheet_2/3v3_esp32
- J6 pad 1: 3.3V -> /chandu_sheet_2/3v3_esp32
- R11 pad 2: 3.3V -> /chandu_sheet_2/3v3_esp32
- R12 pad 2: 3.3V -> /chandu_sheet_2/3v3_esp32
- R_dac1_pup_scl1 pad 2: 3.3V -> /chandu_sheet_2/3v3_esp32
- R_dac1_pup_sda1 pad 1: 3.3V -> /chandu_sheet_2/3v3_esp32
- U2 pad 1: Net-(U2-3V3) -> /chandu_sheet_2/3v3_esp32
- U2 pad 2: Net-(U2-3V3) -> /chandu_sheet_2/3v3_esp32
Routing:
- net /chandu_sheet_2/3v3_esp32: track 0.00 -> 299.6 mm
- net /chandu_sheet_2/\ON_a: track 0.00 -> 246.5 mm
- net 12V: track 30.6 -> 200.7 mm
- net /chandu_sheet_2/vset_b: track 0.00 -> 151.2 mm
- net /chandu_sheet_2/ref_a: track 0.00 -> 108.1 mm
- net /chandu_sheet_2/vset_a: track 0.00 -> 102.5 mm
- net /chandu_sheet_2/\ON_b: track 7.26 -> 103.7 mm
- net /chandu_sheet_2/ref_b: track 0.00 -> 92.1 mm
- net /chandu_sheet_2/adc_I_a: track 0.00 -> 89.0 mm
- net /chandu_sheet_2/adc_V_a: track 0.00 -> 87.1 mm
- net /sunny_sheet_1/v_startup: track 23.7 -> 105.5 mm
- net 3.3V: track 25.7 -> 97.3 mm
- net /chandu_sheet_2/scl_a: track 0.00 -> 55.0 mm
- net Net-(C_filter2-Pad1): track 49.8 -> 101.6 mm
- net GND: track 0.35 -> 51.0 mm, vias 0 -> 16
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- added copper zone on B.Cu, net GND
- added copper zone on F.Cu, net GND
- added copper zone on B.Cu, net GND1
- added copper zone on F.Cu, net GND1
