File: kicad-files/chandra_queenofnight.kicad_pcb (KiCad board)
At the start: 2 copper layers, 242.2 x 183.1 mm, 85 parts, among them IC1 bp060674p12, IC2 bp060674p12, J1 B5B-XH-A_rotataryKnob, J10 51494-2, J3 B5B-XH-A_rotataryKnob, J4 B2B-XH-A__LF__SN_ledTwoTermin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, J5 B2B-XH-A__LF__SN_ledTwoTermin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, J6 B4B-XH-A_LF__SN_oled_display, J8 51494-2, J9 1717732, Q1 FQPF7N90C, T1 7508112339, U10 Optocoupler_DC_PhotoNPN_AKEC, U11 TL431D, U12 ZC576300, U13 ZC576300, U2 DEVKIT_V1_ESP32-WROOM-32, U4 MIC4684, U5 UC3842N, U9 AP2112K-3.3, X1 B2P-VH, X2 B2P-VH, X3 B2P-VH, X4 B2P-VH, X5 B2P-VH

Commit message: Initialtes iprayitworks2
Parts:
- R8: value 20k -> 10k
- renumbered C_decoup_12V2 to C_decoup_12V2?1, C_decoup_3V2 to C_decoup_3V2?1, R11 to R11?1, R12 to R12?1
Connections:
- net Net-(IC1-GND_2) renamed /chandu_sheet_2/hv_-1
- net Net-(IC1-HV) renamed /chandu_sheet_2/hv_+1
- net Net-(IC2-GND_2) renamed /chandu_sheet_2/hv_-2
- net Net-(IC2-HV) renamed /chandu_sheet_2/hv_+2
- C_Y_2 pad 1: /sunny_sheet_1/G -> /sunny_sheet_1/N
- C_Y_2 pad 2: /sunny_sheet_1/N -> /sunny_sheet_1/G
Changed lines of the file:
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@@
 			(layers "*.Cu" "*.Mask")
 			(remove_unused_layers no)
-			(net "Net-(IC1-GND_2)")
+			(net "/chandu_sheet_2/hv_-1")
 			(pinfunction "GND_2_9")
 			(pintype "passive")
@@
 			(layers "*.Cu" "*.Mask")
 			(remove_unused_layers no)
-			(net "Net-(IC1-HV)")
+			(net "/chandu_sheet_2/hv_+1")
 			(pinfunction "HV_10")
 			(pintype "passive")
@@
 			(layers "*.Cu" "*.Mask")
 			(remove_unused_layers no)
-			(net "Net-(IC2-GND_2)")
+			(net "/chandu_sheet_2/hv_-2")
 			(pintype "bidirectional")
 			(solder_mask_margin 0.102)
@@
 			(layers "*.Cu" "*.Mask")
 			(remove_unused_layers no)
-			(net "Net-(IC2-HV)")
+			(net "/chandu_sheet_2/hv_+2")
 			(pintype "bidirectional")
 			(solder_mask_margin 0.102)
@@
 		(descr "Resistor, Axial_DIN0207 series, Axial, Vertical, pin pitch=2.54mm, 0.25W = 1/4W, length*diameter=6.3*2.5mm^2, http://cdn-reichelt.de/documents/datenblatt/B400/1_4W%23YAG.pdf")
 		(tags "Resistor Axial_DIN0207 series Axial Vertical pin pitch 2.54mm 0.25W = 1/4W length 6.3mm diameter 2.5mm")
-		(property "Reference" "R11"
+		(property "Reference" "R11?1"
 			(at 1.27 -2.37 90)
 			(layer "F.SilkS")
@@
 			(layers "*.Cu" "*.Mask")
 			(remove_unused_layers no)
-			(net "Net-(IC1-GND_2)")
+			(net "/chandu_sheet_2/hv_-1")
 			(pintype "bidirectional")
 			(solder_mask_margin 0.102)
@@
 			(layers "*.Cu" "*.Mask")
 			(remove_unused_layers no)
-			(net "Net-(IC1-HV)")
+			(net "/chandu_sheet_2/hv_+1")
 			(pintype "bidirectional")
 			(solder_mask_margin 0.102)
@@
 		(descr "CP, Radial series, Radial, pin pitch=2.00mm, diameter=5mm, height=7mm, Electrolytic Capacitor")
 		(tags "CP Radial series Radial pin pitch 2.00mm diameter 5mm height 7mm Electrolytic Capacitor")
-		(property "Reference" "C_decoup_12V2"
+		(property "Reference" "C_decoup_12V2?1"
 			(at -3.644888 2.6 90)
 			(layer "F.SilkS")
@@
 		(descr "Resistor, Axial_DIN0207 series, Axial, Vertical, pin pitch=2.54mm, 0.25W = 1/4W, length*diameter=6.3*2.5mm^2, http://cdn-reichelt.de/documents/datenblatt/B400/1_4W%23YAG.pdf")
 		(tags "Resistor Axial_DIN0207 series Axial Vertical pin pitch 2.54mm 0.25W = 1/4W length 6.3mm diameter 2.5mm")
-		(property "Reference" "R12"
+		(property "Reference" "R12?1"
 			(at 0.9 2.35 90)
 			(layer "F.SilkS")
@@
 			(layers "*.Cu" "*.Mask")
 			(remove_unused_layers no)
-			(net "/sunny_sheet_1/G")
+			(net "/sunny_sheet_1/N")
 			(pintype "passive")
 		)
@@
 			(layers "*.Cu" "*.Mask")
 			(remove_unused_layers no)
-			(net "/sunny_sheet_1/N")
+			(net "/sunny_sheet_1/G")
 			(pintype "passive")
 		)
@@
 		(descr "CP, Radial series, Radial, pin pitch=2.00mm, diameter=5mm, height=7mm, Electrolytic Capacitor")
 		(tags "CP Radial series Radial pin pitch 2.00mm diameter 5mm height 7mm Electrolytic Capacitor")
-		(property "Reference" "C_decoup_3V2"
+		(property "Reference" "C_decoup_3V2?1"
 			(at 1.1 3.55 0)
 			(layer "F.SilkS")
@@
 			(layers "*.Cu" "*.Mask")
 			(remove_unused_layers no)
-			(net "Net-(IC2-GND_2)")
+			(net "/chandu_sheet_2/hv_-2")
 			(pinfunction "GND_2_9")
 			(pintype "passive")
@@
 			(layers "*.Cu" "*.Mask")
 			(remove_unused_layers no)
-			(net "Net-(IC2-HV)")
+			(net "/chandu_sheet_2/hv_+2")
 			(pinfunction "HV_10")
 			(pintype "passive")
@@
 			)
 		)
-		(property "Value" "20k"
+		(property "Value" "10k"
 			(at 3.81 2.37 90)
 			(layer "F.Fab")
@@
 	)
 	(segment
-		(start 283.931381 69.078001)
-		(end 283.931381 41.681381)
-		(width 0.254)
-		(layer "F.Cu")
-		(net "Net-(IC1-GND_2)")
-	)
-	(segment
-		(start 283.931381 41.681381)
-		(end 278.9 36.65)
-		(width 0.254)
-		(layer "F.Cu")
-		(net "Net-(IC1-GND_2)")
-	)
-	(segment
-		(start 268.691381 69.078001)
-		(end 268.691381 39.441381)
-		(width 0.254)
-		(layer "F.Cu")
-		(net "Net-(IC1-HV)")
-	)
-	(segment
-		(start 268.691381 39.441381)
-		(end 265.9 36.65)
-		(width 0.254)
-		(layer "F.Cu")
-		(net "Net-(IC1-HV)")
-	)
-	(segment
 		(start 303.131381 136.478001)
 		(end 303.131381 128.508001)
@@
 	)
 	(segment
-		(start 327.031381 42.681381)
-		(end 322.4 38.05)
-		(width 0.254)
-		(layer "F.Cu")
-		(net "Net-(IC2-GND_2)")
-	)
-	(segment
-		(start 327.031381 69.078001)
-		(end 327.031381 42.681381)
-		(width 0.254)
-		(layer "F.Cu")
-		(net "Net-(IC2-GND_2)")
-	)
-	(segment
-		(start 311.791381 69.078001)
-		(end 311.791381 40.441381)
-		(width 0.254)
-		(layer "F.Cu")
-		(net "Net-(IC2-HV)")
-	)
-	(segment
-		(start 311.791381 40.441381)
-		(end 309.4 38.05)
-		(width 0.254)
-		(layer "F.Cu")
-		(net "Net-(IC2-HV)")
-	)
-	(segment
 		(start 184.501381 146.788001)
 		(end 177.901381 153.388001)
@@
 		(net "/chandu_sheet_2/v_mon_b")
 	)
+	(segment
+		(start 268.691381 69.078001)
+		(end 268.691381 39.441381)
+		(width 0.254)
+		(layer "F.Cu")
+		(net "/chandu_sheet_2/hv_+1")
+	)
+	(segment
+		(start 268.691381 39.441381)
+		(end 265.9 36.65)
+		(width 0.254)
+		(layer "F.Cu")
+		(net "/chandu_sheet_2/hv_+1")
+	)
+	(segment
+		(start 283.931381 69.078001)
+		(end 283.931381 41.681381)
+		(width 0.254)
+		(layer "F.Cu")
+		(net "/chandu_sheet_2/hv_-1")
+	)
+	(segment
+		(start 283.931381 41.681381)
+		(end 278.9 36.65)
+		(width 0.254)
+		(layer "F.Cu")
+		(net "/chandu_sheet_2/hv_-1")
+	)
+	(segment
+		(start 327.031381 42.681381)
+		(end 322.4 38.05)
+		(width 0.254)
+		(layer "F.Cu")
+		(net "/chandu_sheet_2/hv_-2")
+	)
+	(segment
+		(start 327.031381 69.078001)
+		(end 327.031381 42.681381)
+		(width 0.254)
+		(layer "F.Cu")
+		(net "/chandu_sheet_2/hv_-2")
+	)
+	(segment
+		(start 311.791381 69.078001)
+		(end 311.791381 40.441381)
+		(width 0.254)
+		(layer "F.Cu")
+		(net "/chandu_sheet_2/hv_+2")
+	)
+	(segment
+		(start 311.791381 40.441381)
+		(end 309.4 38.05)
+		(width 0.254)
+		(layer "F.Cu")
+		(net "/chandu_sheet_2/hv_+2")
+	)
 	(zone
