File: kicad-files/chandu.kicad_sch (KiCad schematic)
At the start: 32 parts, among them IC1 bp060674p12, IC2 bp060674p12, J1 B5B-XH-A_rotataryKnob, J10 51494-2, J3 B5B-XH-A_rotataryKnob, J4 B2B-XH-A__LF__SN_ledTwoTermin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, J5 B2B-XH-A__LF__SN_ledTwoTermin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, J6 B4B-XH-A_LF__SN_oled_display, J8 51494-2, U12 ZC576300, U13 ZC576300, U2 DEVKIT_V1_ESP32-WROOM-32, X1 B2P-VH, X3 B2P-VH, X5 B2P-VH

Commit message: Initialtes iprayitworks2
Parts:
- gave numbers to parts that had none: 4
Changed lines of the file:
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@@
 		(dnp no)
 		(fields_autoplaced yes)
-		(property "Reference" "R12??"
+		(property "Reference" "R12?1"
 			(at 207.01 157.48 90)
 			(show_name no)
@@
 			(project "chandra_queenofnight"
 				(path "/fe3f1796-d4c1-46ec-bdb5-a29f35c8d4af/d021fc71-9d18-4a27-819f-074c7472d77d"
-					(reference "R12??")
+					(reference "R12?1")
 					(unit 1)
 				)
@@
 		(dnp no)
 		(fields_autoplaced yes)
-		(property "Reference" "R11??"
+		(property "Reference" "R11?1"
 			(at 194.31 66.04 90)
 			(show_name no)
@@
 			(project "chandra_queenofnight"
 				(path "/fe3f1796-d4c1-46ec-bdb5-a29f35c8d4af/d021fc71-9d18-4a27-819f-074c7472d77d"
-					(reference "R11??")
+					(reference "R11?1")
 					(unit 1)
 				)
@@
 		(dnp no)
 		(fields_autoplaced yes)
-		(property "Reference" "C_decoup_12V2??"
+		(property "Reference" "C_decoup_12V2?1"
 			(at 227.33 81.2799 0)
 			(show_name no)
@@
 			(project "chandra_queenofnight"
 				(path "/fe3f1796-d4c1-46ec-bdb5-a29f35c8d4af/d021fc71-9d18-4a27-819f-074c7472d77d"
-					(reference "C_decoup_12V2??")
+					(reference "C_decoup_12V2?1")
 					(unit 1)
 				)
@@
 		(in_pos_files yes)
 		(dnp no)
-		(property "Reference" "C_decoup_3V2??"
+		(property "Reference" "C_decoup_3V2?1"
 			(at 66.548 71.374 90)
 			(show_name no)
@@
 			(project "chandra_queenofnight"
 				(path "/fe3f1796-d4c1-46ec-bdb5-a29f35c8d4af/d021fc71-9d18-4a27-819f-074c7472d77d"
-					(reference "C_decoup_3V2??")
+					(reference "C_decoup_3V2?1")
 					(unit 1)
 				)
