File: kicad-files/sunny.kicad_sch (KiCad schematic)
At the start: 53 parts, among them J9 1717732, Q1 FQPF7N90C, T1 7508112339, U10 Optocoupler_DC_PhotoNPN_AKEC, U11 TL431D, U4 MIC4684, U5 UC3842N, U9 AP2112K-3.3, X2 B2P-VH, X4 B2P-VH

Commit message: Initialtes iprayitworks2
Connections:
- net G: now also C_Y_2.2; no longer C_Y_2.1
- net N: now also C_Y_2.1; no longer C_Y_2.2
Other:
- note added: "100u"
- note added: "1uF"
- moved on the sheet: C_Y_2, D3, RV1, TH1
